Commit message: fix: windows forward slash issue

File: tests/data/assembly_expected.urdf (robot description, URDF)
Before this commit: robot test_robot, 9 links, 8 joints
Links:
- link Assembly_2_1_Assembly_1_1_Part_10_1: geometry collision mesh filename=meshes/Assembly_2_1_Assembly_1_1_Part_10_1.stl; visual mesh filename=meshes/Assembly_2_1_Assembly_1_1_Part_10_1.stl
- link Assembly_2_1_Assembly_1_1_Part_4_1: geometry collision mesh filename=meshes/Assembly_2_1_Assembly_1_1_Part_4_1.stl; visual mesh filename=meshes/Assembly_2_1_Assembly_1_1_Part_4_1.stl
- link Assembly_2_1_Assembly_1_2_Part_10_1: geometry collision mesh filename=meshes/Assembly_2_1_Assembly_1_2_Part_10_1.stl; visual mesh filename=meshes/Assembly_2_1_Assembly_1_2_Part_10_1.stl
- link Assembly_2_1_Assembly_1_2_Part_4_1: geometry collision mesh filename=meshes/Assembly_2_1_Assembly_1_2_Part_4_1.stl; visual mesh filename=meshes/Assembly_2_1_Assembly_1_2_Part_4_1.stl
- link Assembly_2_1_Part_12_1: geometry collision mesh filename=meshes/Assembly_2_1_Part_12_1.stl; visual mesh filename=meshes/Assembly_2_1_Part_12_1.stl
- link Assembly_2_1_Part_6_1: geometry collision mesh filename=meshes/Assembly_2_1_Part_6_1.stl; visual mesh filename=meshes/Assembly_2_1_Part_6_1.stl
- link Part_14_1: geometry collision mesh filename=meshes/Part_14_1.stl; visual mesh filename=meshes/Part_14_1.stl
- link Part_15_1: geometry collision mesh filename=meshes/Part_15_1.stl; visual mesh filename=meshes/Part_15_1.stl
- link Part_1_1: geometry collision mesh filename=meshes/Part_1_1.stl; visual mesh filename=meshes/Part_1_1.stl
